File: Encoder_SPI_A1333/Encoder_SPI_A1333.kicad_pcb (KiCad board)
At the start: 2 copper layers, 21 x 17 mm, 10 parts, among them J1 Conn_01x06_MountingPin, J2 Castellations_ABI, U1 A1333

Commit message: A1334 encoder design first production run
Other:
- net class Default removed
