File: Encoder_SPI_MA730/Encoder_SPI_MA730.kicad_pcb (KiCad board)
At the start: 2 copper layers, 21 x 10 mm, 13 parts, among them J1 Conn_01x06_MountingPin, J2 Castellations_ABI, U1 MA730

Commit message: new encoder models, updated READMEs
Other:
- net class Default removed
