File: Encoder_SPI_MA330/Encoder_SPI_MA330.kicad_sch (KiCad schematic)
At the start: 9 parts, among them J1 Conn_01x06_MountingPin, J2 Castellations_ABI, U1 MA730

Commit message: update labels
Parts:
- U1: value MA730 -> MA330
Changed lines of the file:
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@@
     (in_bom yes) (on_board yes)
     (property "Reference" "U1" (id 0) (at 120.65 71.12 0))
-    (property "Value" "MA730" (id 1) (at 137.16 71.12 0))
+    (property "Value" "MA330" (id 1) (at 137.16 71.12 0))
     (property "Footprint" "Package_DFN_QFN:QFN-16-1EP_3x3mm_P0.5mm_EP1.75x1.75mm" (id 2) (at 129.54 106.68 0)
       (effects (font (size 1.27 1.27)) hide)
@@
     )
     (path "/00000000-0000-0000-0000-0000606d7b3d"
-      (reference "U1") (unit 1) (value "MA730") (footprint "Package_DFN_QFN:QFN-16-1EP_3x3mm_P0.5mm_EP1.75x1.75mm")
+      (reference "U1") (unit 1) (value "MA330") (footprint "Package_DFN_QFN:QFN-16-1EP_3x3mm_P0.5mm_EP1.75x1.75mm")
     )
   )
