File: Encoder_SPI_MT6701/Encoder_SPI_MT6701.kicad_sch (KiCad schematic)
At the start: 11 parts, among them J1 Conn_01x06_MountingPin, J2 Conn_01x02, SW1 SW_DIP_x01, U1 MT6701QT

Commit message: update labels
Parts:
- J1: Port SPI -> SSI / I2C / ABZ
Other:
- note added: "(ABZ: A, I2C: SDA)"
- note added: "(ABZ: B, I2C: SCL)"
- note added: "(ABZ: Z, I2C: pull high to VCC)"
Changed lines of the file:
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@@
     (stroke (width 0) (type default) (color 0 0 0 0))
+  )
+  (text "(ABZ: A, I2C: SDA)" (at 81.28 83.82 0)
+    (effects (font (size 1.27 1.27)) (justify left bottom))
+  )
+  (text "(ABZ: Z, I2C: pull high to VCC)" (at 81.28 88.9 0)
+    (effects (font (size 1.27 1.27)) (justify left bottom))
+  )
+  (text "(ABZ: B, I2C: SCL)" (at 81.28 86.36 0)
+    (effects (font (size 1.27 1.27)) (justify left bottom))
   )
   (text "Mode has internal 200kΩ pullup.\nMODE==0 ABZ mode\nMODE==1 SSI/I2C mode"
@@
   (symbol (lib_id "Connector_Generic_MountingPin:Conn_01x06_MountingPin") (at 69.85 81.28 0) (mirror y) (unit 1)
     (in_bom yes) (on_board yes)
-    (property "Reference" "J1" (id 0) (at 69.85 71.12 0))
+    (property "Reference" "J1" (id 0) (at 69.85 73.025 0))
     (property "Value" "Conn_01x06_MountingPin" (id 1) (at 67.6148 85.7758 0)
       (effects (font (size 1.27 1.27)) (justify left) hide)
@@
       (effects (font (size 1.27 1.27)) hide)
     )
-    (property "Port" "SPI" (id 4) (at 69.85 73.66 0))
+    (property "Port" "SSI / I2C / ABZ" (id 4) (at 58.42 82.55 0))
     (property "Manu" "Scondar Electronic Limited" (id 5) (at 69.85 81.28 0)
       (effects (font (size 1.27 1.27)) hide)
