File: Encoder_SPI_MT6701_I2CAdapter/Encoder_SPI_MT6701_I2CAdapter.kicad_sch (KiCad schematic)
At the start: 21 parts, among them J1 3.3V in, J2 JST_SH_SM04B, J3 5V in, J4 JST_SH_SM06B, U1 NXB0102GTX

Commit message: fix incorrect footprint
Connections:
- net MISO: now also U1.8 (B1); no longer U1.1 (B2)
- net SCK: now also U1.1 (B2); no longer U1.8 (B1)
- net SCL_A: now also U1.4 (A2); no longer U1.5 (A1)
- net SDA_A: now also U1.5 (A1); no longer U1.4 (A2)
Changed lines of the file:
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@@
     (effects (font (size 1.27 1.27)) (justify left bottom))
   )
-  (label "SDA_A" (at 127 102.87 180)
+  (label "SDA_A" (at 127 100.33 180)
     (effects (font (size 1.27 1.27)) (justify right bottom))
   )
@@
     (effects (font (size 1.27 1.27)) (justify left bottom))
   )
-  (label "SCL_A" (at 127 100.33 180)
+  (label "SCL_A" (at 127 102.87 180)
     (effects (font (size 1.27 1.27)) (justify right bottom))
   )
@@
     (effects (font (size 1.27 1.27)) (justify left bottom))
   )
-  (label "SCL_B" (at 147.32 100.33 0)
+  (label "SCL_B" (at 147.32 102.87 0)
     (effects (font (size 1.27 1.27)) (justify left bottom))
   )
-  (label "SDA_B" (at 147.32 102.87 0)
+  (label "SDA_B" (at 147.32 100.33 0)
     (effects (font (size 1.27 1.27)) (justify left bottom))
   )

Commit message: add 3d models, fix bugs
Parts:
- U1: value NXB0102GTX -> NXS0102GT; Part NXB0102GTX -> NXS0102GT
Changed lines of the file:
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@@
       (effects (font (size 1.27 1.27)) (justify left))
     )
-    (property "Value" "NXB0102GTX" (id 1) (at 137.16 111.76 0)
+    (property "Value" "NXS0102GT" (id 1) (at 137.16 111.76 0)
       (effects (font (size 1.27 1.27)) (justify left))
     )
@@
       (effects (font (size 1.27 1.27)) hide)
     )
-    (property "Part" "NXB0102GTX" (id 5) (at 137.16 100.33 0)
+    (property "Part" "NXS0102GT" (id 5) (at 137.16 100.33 0)
       (effects (font (size 1.27 1.27)) hide)
     )
@@
     )
     (path "/3f86c136-a6a0-44e4-98c5-ec3baf86fdf4"
-      (reference "U1") (unit 1) (value "NXB0102GTX") (footprint "runger:SOT833-1 (XSON8)")
-    )
-  )
+      (reference "U1") (unit 1) (value "NXS0102GT") (footprint "runger:SOT833-1 (XSON8)")
+    )
+  )
