File: Encoder_MT6835/Encoder_MT6835.kicad_pcb (KiCad board)
At the start: 2 copper layers, 21 x 17 mm, 11 parts, among them J1 Conn_01x06_MountingPin, J2 Pad_OUT, J3 Conn_01x06_MountingPin, U1 MT6835

Commit message: production v1
Parts:
- C1: moved to B.Cu
- moved C1 4.67 mm to (120.5, 93.8), turned to 180 degrees
Routing:
- net GND: track 18.1 -> 21.6 mm
- net VCC: track 24.2 -> 27.3 mm, vias 0 -> 1
