File: Encoder_SPI_AS5047P_big/Encoder_SPI_AS5047P.kicad_sch (KiCad schematic)
At the start: 13 parts, among them J1 Conn_01x06_MountingPin, J2 Conn_01x06_MountingPin, T1 Tab, T2 Tab, U2 AS5047D

Commit message: encoder updates
Parts:
- C1: Manu (none) -> Generic; Notes (none) -> eg. YAGEO CC0603KRX7R6BB105; Part (none) -> 1uF 10V
- C2: Manu (none) -> Generic; Notes (none) -> eg. YAGEO CC0603KRX7R6BB104; Part (none) -> 100nF 10V
- D1: Manu (none) -> Generic; Notes inexpensive green LED please -> e.g. XINGLIGHT XL-2012UGC; Part (none) -> Green LED
- H1, H2, JP1: now left out of the parts list
- J1, J2: Notes JST SH_SM06B-SRSS-TB_1x06-1MP_P1.00mm_Horizontal or compati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 -> compatible to JST SH_SM06B-SRSS-TB_1x06-1MP_P1.00mm_Horizon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
- U2: Manu (none) -> AMS; Notes (none) -> Depends on price also: AS5047P-ATSM; Part (none) -> AS5047U-HTSM or
